File: 40% with arrows.sch (KiCad schematic (older format))
At the start: 117 parts, among them J1 USB_C_Receptacle_USB2.0, K1 KEYSW, K10 KEYSW, K11 KEYSW, K12 KEYSW, K13 KEYSW, K14 KEYSW, K15 KEYSW, K16 KEYSW, K17 KEYSW, K18 KEYSW, K19 KEYSW, K2 KEYSW, K20 KEYSW, K21 KEYSW, K22 KEYSW, K23 KEYSW, K24 KEYSW, K25 KEYSW, K26 KEYSW, K27 KEYSW, K28 KEYSW, K29 KEYSW, K3 KEYSW, K30 KEYSW, K31 KEYSW, K32 KEYSW, K33 KEYSW, K34 KEYSW, K35 KEYSW, K36 KEYSW, K37 KEYSW, K38 KEYSW, K39 KEYSW, K4 KEYSW, K40 KEYSW, K41 KEYSW, K42 KEYSW, K43 KEYSW, K44 KEYSW, K45 KEYSW, K46 KEYSW, K47 KEYSW, K48 KEYSW, K49 KEYSW, K5 KEYSW, K6 KEYSW, K7 KEYSW, K8 KEYSW, K9 KEYSW, SW1 SW_PUSH, U1 ATMEGA32U4, Y1 Crystal_GND24

Commit message: Changes to the pcb and schematic
Changes to the pcb and schematic by the advice of Taylor.
Parts:
- F1: footprint Fuse:Fuse_0402_1005Metric -> Fuse:Fuse_0603_1608Metric
Changed lines of the file:
@@
 F 0 "F1" V 2050 8050 50  0000 C CNN
 F 1 "Fuse" V 2150 8050 50  0000 C CNN
-F 2 "Fuse:Fuse_0402_1005Metric" V 2080 8050 50  0001 C CNN
+F 2 "Fuse:Fuse_0603_1608Metric" V 2080 8050 50  0001 C CNN
 F 3 "~" H 2150 8050 50  0001 C CNN
 	1    2150 8050
