File: 40% with arrows.kicad_pcb (KiCad board)
At the start: 2 copper layers, 268 x 82.2 mm, 114 parts, among them K1 KEYSW, K10 KEYSW, K11 KEYSW, K12 KEYSW, K13 KEYSW, K14 KEYSW, K15 KEYSW, K16 KEYSW, K17 KEYSW, K18 KEYSW, K19 KEYSW, K2 KEYSW, K20 KEYSW, K21 KEYSW, K22 KEYSW, K23 KEYSW, K24 KEYSW, K25 KEYSW, K26 KEYSW, K27 KEYSW, K28 KEYSW, K29 KEYSW, K3 KEYSW, K30 KEYSW, K31 KEYSW, K32 KEYSW, K33 KEYSW, K34 KEYSW, K35 KEYSW, K36 KEYSW, K37 KEYSW, K38 KEYSW, K39 KEYSW, K4 KEYSW, K40 KEYSW, K41 KEYSW, K42 KEYSW, K43 KEYSW, K44 KEYSW, K45 KEYSW, K46 KEYSW, K47 KEYSW, K48 KEYSW, K49 KEYSW, K5 KEYSW, K6 KEYSW, K7 KEYSW, K8 KEYSW, K9 KEYSW, P1 USB_C_Plug_USB2.0, SW1 SW_PUSH, U1 ATMEGA32U4, X1 XTAL_GND

Commit message: Changes to the pcb and schematic
Changes to the pcb and schematic by the advice of Taylor.
Parts:
- removed P1: USB_C_Plug_USB2.0, Connector_USB:USB_C_Receptacle_Palconn_UTC16-G
- removed X1: XTAL_GND, Crystal:Crystal_SMD_SeikoEpson_FA238-4Pin_3.2x2.5mm_HandSoldering
- added F1: Fuse, Fuse:Fuse_0603_1608Metric, B.Cu at (244.8, 45.3)
- added J1: USB_C_Receptacle_USB2.0, Connector_USB:USB_C_Receptacle_Palconn_UTC16-G, B.Cu at (249.9, 39.4)
- added R5: 5.1k, Resistor_SMD:R_0402_1005Metric, B.Cu at (251.7, 47.4)
- added R6: 5.1k, Resistor_SMD:R_0402_1005Metric, B.Cu at (247.9, 47.3)
- added Y1: Crystal_GND24, Crystal:Crystal_SMD_SeikoEpson_FA238-4Pin_3.2x2.5mm, B.Cu at (142.6, 103.6)
- C2, C3: value 22p -> 22pF
- C4, C5, C6, C7, C8: moved to F.Cu
- moved C8 15.1 mm to (132.2, 100.5)
- moved C6 15.0 mm to (130.3, 100.1), turned to 180 degrees
- moved C7 11.0 mm to (135.8, 101.7), turned to 0 degrees
- moved C5 10.2 mm to (130.3, 106.5), turned to 180 degrees
- moved C4 4.72 mm to (137.1, 106.0), turned to 270 degrees
- moved C3 1.98 mm to (142.6, 106.4), turned to 0 degrees
- moved C2 1.96 mm to (142.7, 100.8)
Connections:
- K14 pad 1: Net-(K1-Pad1) -> Net-(K14-Pad1)
- K15 pad 1: Net-(K2-Pad1) -> Net-(K15-Pad1)
- K16 pad 1: Net-(K3-Pad1) -> Net-(K16-Pad1)
- K17 pad 1: Net-(K4-Pad1) -> Net-(K17-Pad1)
- K18 pad 1: Net-(K5-Pad1) -> Net-(K18-Pad1)
- K19 pad 1: Net-(K6-Pad1) -> Net-(K19-Pad1)
- K20 pad 1: Net-(K7-Pad1) -> Net-(K20-Pad1)
- K21 pad 1: Net-(K8-Pad1) -> Net-(K21-Pad1)
- K22 pad 1: Net-(K9-Pad1) -> Net-(K22-Pad1)
- K23 pad 1: Net-(K10-Pad1) -> Net-(K23-Pad1)
- K24 pad 1: Net-(K11-Pad1) -> Net-(K24-Pad1)
- K25 pad 1: Net-(K12-Pad1) -> Net-(K25-Pad1)
- K26 pad 1: Net-(K13-Pad1) -> Net-(K26-Pad1)
- K27 pad 1: Net-(K1-Pad1) -> Net-(K27-Pad1)
- K28 pad 1: Net-(K2-Pad1) -> Net-(K28-Pad1)
- K29 pad 1: Net-(K3-Pad1) -> Net-(K29-Pad1)
- K30 pad 1: Net-(K4-Pad1) -> Net-(K30-Pad1)
- K31 pad 1: Net-(K5-Pad1) -> Net-(K31-Pad1)
- K32 pad 1: Net-(K6-Pad1) -> Net-(K32-Pad1)
- K33 pad 1: Net-(K7-Pad1) -> Net-(K33-Pad1)
- K34 pad 1: Net-(K8-Pad1) -> Net-(K34-Pad1)
- K35 pad 1: Net-(K9-Pad1) -> Net-(K35-Pad1)
- K36 pad 1: Net-(K10-Pad1) -> Net-(K36-Pad1)
- K37 pad 1: Net-(K11-Pad1) -> Net-(K37-Pad1)
- K38 pad 1: Net-(K12-Pad1) -> Net-(K38-Pad1)
- K39 pad 1: Net-(K13-Pad1) -> Net-(K39-Pad1)
- K40 pad 1: Net-(K1-Pad1) -> Net-(K40-Pad1)
- K41 pad 1: Net-(K2-Pad1) -> Net-(K41-Pad1)
- K42 pad 1: Net-(K3-Pad1) -> Net-(K42-Pad1)
- K43 pad 1: Net-(K4-Pad1) -> Net-(K43-Pad1)
- K44 pad 1: Net-(K7-Pad1) -> Net-(K44-Pad1)
- K45 pad 1: Net-(K9-Pad1) -> Net-(K45-Pad1)
- K46 pad 1: Net-(K10-Pad1) -> Net-(K46-Pad1)
- K47 pad 1: Net-(K11-Pad1) -> Net-(K47-Pad1)
- K48 pad 1: Net-(K12-Pad1) -> Net-(K48-Pad1)
- K49 pad 1: Net-(K13-Pad1) -> Net-(K49-Pad1)
- U1 pad 10: Net-(D1-Pad1) -> Net-(U1-Pad10)
- U1 pad 11: Net-(D40-Pad1) -> Net-(U1-Pad11)
- U1 pad 25: Net-(K7-Pad1) -> Net-(U1-Pad25)
- U1 pad 26: Net-(K8-Pad1) -> Net-(U1-Pad26)
- U1 pad 27: Net-(K9-Pad1) -> Net-(U1-Pad27)
- U1 pad 28: Net-(K10-Pad1) -> Net-(U1-Pad28)
- U1 pad 29: Net-(K11-Pad1) -> Net-(U1-Pad29)
- U1 pad 30: Net-(K12-Pad1) -> Net-(U1-Pad30)
- U1 pad 31: Net-(K13-Pad1) -> Net-(U1-Pad31)
- U1 pad 36: Net-(K4-Pad1) -> Net-(U1-Pad36)
- U1 pad 37: Net-(K3-Pad1) -> Net-(U1-Pad37)
- U1 pad 38: Net-(K2-Pad1) -> Net-(U1-Pad38)
- U1 pad 39: Net-(K1-Pad1) -> Net-(U1-Pad39)
- U1 pad 40: Net-(K5-Pad1) -> Net-(U1-Pad40)
- U1 pad 41: Net-(K6-Pad1) -> Net-(U1-Pad41)
- U1 pad 8: Net-(D27-Pad1) -> Net-(U1-Pad8)
- U1 pad 9: Net-(D14-Pad1) -> Net-(U1-Pad9)
Routing:
- net VCC: track 43.4 -> 55.7 mm, vias 4 -> 5
- net Net-(F1-Pad1): track 199.5 -> 189.5 mm
- net Net-(F1-Pad2): track 0.00 -> 8.73 mm
- net +5V: track 270.8 -> 276.8 mm, vias 2 -> 9
- net Net-(C3-Pad1): track 11.5 -> 5.51 mm
- net Net-(J1-PadA5): track 0.00 -> 5.30 mm
- net Net-(J1-PadB5): track 0.00 -> 4.99 mm
- net Net-(R1-Pad1): track 189.1 -> 192.4 mm
- net Net-(R2-Pad1): track 191.9 -> 194.3 mm
- net Net-(C2-Pad1): track 9.59 -> 7.91 mm

Commit message: new thinges
Parts:
- moved F1 2.72 mm to (244.8, 48.0)
- moved R1 2.08 mm to (250.6, 47.4)
- moved R2 2.07 mm to (249.2, 47.4)
- moved J1 2.06 mm to (249.9, 41.4)
Connections:
- U1 pad 25: Net-(U1-Pad25) -> Net-(K7-Pad1)
- U1 pad 26: Net-(U1-Pad26) -> Net-(K8-Pad1)
- U1 pad 27: Net-(U1-Pad27) -> Net-(K9-Pad1)
- U1 pad 28: Net-(U1-Pad28) -> Net-(K10-Pad1)
- U1 pad 29: Net-(U1-Pad29) -> Net-(K11-Pad1)
- U1 pad 30: Net-(U1-Pad30) -> Net-(K12-Pad1)
- U1 pad 31: Net-(U1-Pad31) -> Net-(K13-Pad1)
Routing:
- net +5V: track 276.8 -> 268.8 mm
- net Net-(D40-Pad1): track 404.1 -> 399.3 mm
- net Net-(K9-Pad1): track 129.2 -> 125.2 mm
- net Net-(K11-Pad1): track 170.3 -> 166.3 mm
- net Net-(K12-Pad1): track 192.6 -> 188.6 mm
- net Net-(K7-Pad1): track 93.9 -> 90.0 mm
- net Net-(K8-Pad1): track 102.7 -> 98.8 mm
- net Net-(K13-Pad1): track 208.4 -> 204.5 mm
- net Net-(K10-Pad1): track 151.6 -> 147.7 mm
- net Net-(F1-Pad1): track 189.5 -> 186.5 mm
- net Net-(R2-Pad1): track 194.3 -> 192.3 mm
- net Net-(J1-PadA5): track 5.30 -> 3.24 mm
- net Net-(R1-Pad1): track 192.4 -> 190.3 mm
- net Net-(J1-PadB5): track 4.99 -> 2.94 mm
- net Net-(F1-Pad2): track 8.73 -> 9.39 mm
Other:
- board size 268 x 82.2 mm -> 262 x 76.7 mm
